Commit message: nav2-init

File: install/agv_bot/share/agv_bot/models/agv_bot_v1.urdf (robot description, URDF)
Before this commit: robot agv_bot, 5 links, 4 joints
Links:
- added link lidar_link, mass 0.114; collision cylinder length=0.08 radius=0.0508; visual cylinder length=0.08 radius=0.0508
Joints:
- added joint lidar_joint: type fixed, parent base_link, child lidar_link, origin xyz=0.215 0 0.13 rpy=0 0 0
